File: imxrt1011_feather.kicad_pcb (KiCad board)
At the start: 4 copper layers, 50.8 x 22.9 mm, 85 parts, among them J1 Conn_Battery, J2 USB_C_Receptacle_USB2.0, J3 Conn_Left, J4 Conn_Right, Q1 BSS84, SW1 SW_RST, U1 AP2112K-3.3, U2 MCP73831, U3 ESP32-PICO-D4, U4 S25FL064LABNFI04x, U5 MIMXRT1011DAE5A, Y1 24MHz

Commit message: Rev 1
Other:
- board text added: "MIMXRT1011 500MHz • 3.3V 8MB FLASH 128 KB RAM"
- board text removed: "MIMXRT1011 500MHz • 3.3V 16MB FLASH 128 KB RAM"
Changed lines of the file:
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@@
-(kicad_pcb (version 20190907) (host pcbnew "(5.99.0-290-g56525296b)")
+(kicad_pcb (version 20190907) (host pcbnew "(5.99.0-380-g9a82bc396)")
   (general
     (thickness 1.6)
@@
       (layer "F.SilkS" (type "Top Silk Screen"))
       (layer "F.Paste" (type "Top Solder Paste"))
-      (layer "F.Mask" (type "Top Solder Mask") (thickness 0.01) (color "Green"))
+      (layer "F.Mask" (type "Top Solder Mask") (color "Green") (thickness 0.01))
       (layer "F.Cu" (type "copper") (thickness 0.035))
       (layer "dielectric 1" (type "core") (thickness 0.48) (material "FR4") (epsilon_r 4.5) (loss_tangent 0.02))
@@
       (layer "dielectric 3" (type "core") (thickness 0.48) (material "FR4") (epsilon_r 4.5) (loss_tangent 0.02))
       (layer "B.Cu" (type "copper") (thickness 0.035))
-      (layer "B.Mask" (type "Bottom Solder Mask") (thickness 0.01) (color "Green"))
+      (layer "B.Mask" (type "Bottom Solder Mask") (color "Green") (thickness 0.01))
       (layer "B.Paste" (type "Bottom Solder Paste"))
       (layer "B.SilkS" (type "Bottom Silk Screen"))
@@
     (solder_mask_min_width 0.25)
     (aux_axis_origin 0 0)
-    (visible_elements 7FF7FF5F)
+    (visible_elements 7FFFFF5F)
     (pcbplotparams
       (layerselection 0x010fc_ffffffff)
-      (usegerberextensions false)
+      (usegerberextensions true)
       (usegerberattributes false)
       (usegerberadvancedattributes false)
@@
       (outputformat 1)
       (mirror false)
-      (drillshape 1)
+      (drillshape 0)
       (scaleselection 1)
-      (outputdirectory "")
+      (outputdirectory "gerb/")
     )
   )
@@
     (effects (font (size 0.85 0.85) (thickness 0.15)) (justify mirror))
   )
-  (gr_text "MIMXRT1011\n500MHz • 3.3V\n16MB FLASH\n128 KB RAM" (at 184.4 96.7 90) (layer "B.SilkS")
+  (gr_text "MIMXRT1011\n500MHz • 3.3V\n8MB FLASH\n128 KB RAM" (at 184.4 96.7 90) (layer "B.SilkS")
     (effects (font (size 0.85 0.85) (thickness 0.15)) (justify mirror))
   )
