File: feather_mimxrt1011.kicad_pcb (KiCad board)
At the start: 4 copper layers, 50.8 x 22.9 mm, 85 parts, among them J1 Conn_Battery, J2 USB_C_Receptacle_USB2.0, J3 Conn_Left, J4 Conn_Right, Q1 BSS84, SW1 SW_RST, U1 AP2112K-3.3, U2 MCP73831, U3 ESP32-PICO-D4, U4 S25FL064LABNFI04x, U5 MIMXRT1011DAE5A, Y1 24MHz

Commit message: Rev 2
Parts:
- removed C13, C15, C20: 0.1uF, Capacitor_SMD:C_0402_1005Metric
- removed JP1: JP_BOOT_MODE_00, Jumper_Extra:SolderJumper-3_P1.3mm_Bridged12_RoundedPad1.0x1.5mm
- removed JP2: JP_BOOT_MODE_01, Jumper_Extra:SolderJumper-3_P1.3mm_Bridged12_RoundedPad1.0x1.5mm
- removed JP3: JP_CFG00, Jumper_Extra:SolderJumper-3_P1.3mm_Bridged12_RoundedPad1.0x1.5mm
- removed JP4: JP_CFG01, Jumper_Extra:SolderJumper-3_P1.3mm_Bridged12_RoundedPad1.0x1.5mm
- removed JP5: JP_CFG02, Jumper_Extra:SolderJumper-3_P1.3mm_Bridged12_RoundedPad1.0x1.5mm
- removed JP6: JP_CFG03, Jumper_Extra:SolderJumper-3_P1.3mm_Bridged12_RoundedPad1.0x1.5mm
- moved G*** 12.4 mm to (164.1, 93.2)
- moved C14 1.40 mm to (173.8, 97.8)
- moved R12 1.00 mm to (173.8, 94.4)
Connections:
- D4 pad 1: Net-(D4-Pad1) -> (no net)
- J2 pad A8: Net-(J2-PadA8) -> (no net)
- J2 pad B8: Net-(J2-PadB8) -> (no net)
- R10 pad 2: +3V3 -> Net-(C1-Pad1)
- U1 pad 4: Net-(U1-Pad4) -> (no net)
- U3 pad 10: Net-(U3-Pad10) -> (no net)
- U3 pad 11: Net-(U3-Pad11) -> (no net)
- U3 pad 12: Net-(U3-Pad12) -> (no net)
- U3 pad 14: Net-(U3-Pad14) -> (no net)
- U3 pad 15: Net-(U3-Pad15) -> (no net)
- U3 pad 16: Net-(U3-Pad16) -> (no net)
- U3 pad 18: Net-(U3-Pad18) -> (no net)
- U3 pad 20: Net-(U3-Pad20) -> (no net)
- U3 pad 21: Net-(U3-Pad21) -> (no net)
- U3 pad 22: Net-(U3-Pad22) -> (no net)
- U3 pad 24: Net-(U3-Pad24) -> (no net)
- U3 pad 25: Net-(U3-Pad25) -> (no net)
- U3 pad 26: Net-(U3-Pad26) -> (no net)
- U3 pad 27: Net-(U3-Pad27) -> (no net)
- U3 pad 28: Net-(U3-Pad28) -> (no net)
- U3 pad 29: Net-(U3-Pad29) -> (no net)
- U3 pad 30: Net-(U3-Pad30) -> (no net)
- U3 pad 31: Net-(U3-Pad31) -> (no net)
- U3 pad 32: Net-(U3-Pad32) -> (no net)
- U3 pad 33: Net-(U3-Pad33) -> (no net)
- U3 pad 38: Net-(U3-Pad38) -> (no net)
- U3 pad 39: Net-(U3-Pad39) -> (no net)
- U3 pad 42: Net-(U3-Pad42) -> (no net)
- U3 pad 44: Net-(U3-Pad44) -> (no net)
- U3 pad 45: Net-(U3-Pad45) -> (no net)
- U3 pad 47: Net-(U3-Pad47) -> (no net)
- U3 pad 48: Net-(U3-Pad48) -> (no net)
- U3 pad 5: Net-(U3-Pad5) -> (no net)
- U3 pad 6: Net-(U3-Pad6) -> (no net)
- U3 pad 7: Net-(U3-Pad7) -> (no net)
- U3 pad 8: Net-(U3-Pad8) -> (no net)
- U5 pad 21: Net-(U5-Pad21) -> (no net)
- U5 pad 24: /EN -> (no net)
- U5 pad 28: Net-(U5-Pad28) -> (no net)
- U5 pad 36: Net-(U5-Pad36) -> (no net)
- U5 pad 61: /IMXRT1011/BT_CFG03 -> GND
- U5 pad 62: Net-(U5-Pad62) -> (no net)
- U5 pad 72: /IMXRT1011/BOOT_MODE00 -> GND
- U5 pad 73: /IMXRT1011/BOOT_MODE01 -> +3V3
- U5 pad 74: /IMXRT1011/BT_CFG00 -> GND
- U5 pad 75: /IMXRT1011/BT_CFG01 -> GND
- U5 pad 76: /IMXRT1011/BT_CFG02 -> GND
Routing:
- net +3V3: track 79.1 -> 64.1 mm, vias 23 -> 22
- net /IMXRT1011/BT_CFG03: track 10.9 -> 0.00 mm, vias 1 -> 0
- net /IMXRT1011/BT_CFG00: track 9.07 -> 0.00 mm, vias 1 -> 0
- net /IMXRT1011/BOOT_MODE01: track 8.95 -> 0.00 mm, vias 1 -> 0
- net /IMXRT1011/BOOT_MODE00: track 6.76 -> 0.00 mm, vias 1 -> 0
- net /IMXRT1011/BT_CFG01: track 6.70 -> 0.00 mm, vias 1 -> 0
- net /EN: track 30.0 -> 23.3 mm, vias 4 -> 3
- net GND: track 98.4 -> 92.0 mm
- net /~RST~: track 33.3 -> 27.0 mm, vias 2 -> 3
- net Net-(C1-Pad1): track 9.62 -> 15.0 mm, vias 0 -> 2
- net /IMXRT1011/BT_CFG02: track 4.33 -> 0.00 mm, vias 1 -> 0
- net VBUS: track 62.6 -> 61.4 mm, vias 5 -> 6
Other:
- board text added: "Jan 2020"
- board text removed: "BOOT0"
- board text removed: "BOOT1"
- board text removed: "CFG0"
- board text removed: "CFG1"
- board text removed: "CFG2"
- board text removed: "CFG3"
- board text removed: "Nov 2019"
- board text removed: "by arturo182 Nov 2019"
