File: feather_mimxrt1011.sch (KiCad schematic (older format))
At the start: 25 parts, among them J1 Conn_Battery, J2 USB_C_Receptacle_USB2.0, J3 Conn_Left, J4 Conn_Right, Q1 BSS84, SW1 SW_RST, U1 AP2112K-3.3, U2 MCP73831

Commit message: Rev 2
Parts:
- added R10: 100K, Resistor_SMD:R_0402_1005Metric, symbol Device:R_Small
Connections:
- net EN: now also R10.1
- net at C1.1, D1.1 (K), Q1.2 (S)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: now also R10.2
Other:
- moved on the sheet: C2, TP3, TP4, U1
