File: imxrt1011.sch (KiCad schematic (older format))
At the start: 45 parts, among them U4 S25FL064LABNFI04x, U5 MIMXRT1011DAE5A, Y1 24MHz

Commit message: Rev 2
Parts:
- removed C13, C15, C20: 0.1uF, Capacitor_SMD:C_0402_1005Metric, symbol Device:C_Small
- removed JP1: JP_BOOT_MODE_00, Jumper_Extra:SolderJumper-3_P1.3mm_Bridged12_RoundedPad1.0x1.5mm, symbol Jumper:SolderJumper_3_Bridged12
- removed JP2: JP_BOOT_MODE_01, Jumper_Extra:SolderJumper-3_P1.3mm_Bridged12_RoundedPad1.0x1.5mm, symbol Jumper:SolderJumper_3_Bridged12
- removed JP3: JP_CFG00, Jumper_Extra:SolderJumper-3_P1.3mm_Bridged12_RoundedPad1.0x1.5mm, symbol Jumper:SolderJumper_3_Bridged12
- removed JP4: JP_CFG01, Jumper_Extra:SolderJumper-3_P1.3mm_Bridged12_RoundedPad1.0x1.5mm, symbol Jumper:SolderJumper_3_Bridged12
- removed JP5: JP_CFG02, Jumper_Extra:SolderJumper-3_P1.3mm_Bridged12_RoundedPad1.0x1.5mm, symbol Jumper:SolderJumper_3_Bridged12
- removed JP6: JP_CFG03, Jumper_Extra:SolderJumper-3_P1.3mm_Bridged12_RoundedPad1.0x1.5mm, symbol Jumper:SolderJumper_3_Bridged12
- removed R10: 100K, Resistor_SMD:R_0402_1005Metric, symbol Device:R_Small
Connections:
- net BOOT_MODE00 is gone; now on net GND: U5.72 (GPIO_SD_04)
- net BOOT_MODE01 is gone; now on net +3V3: U5.73 (GPIO_SD_03)
- net BT_CFG00 is gone; now on net GND: U5.74 (GPIO_SD_02)
- net BT_CFG01 is gone; now on net GND: U5.75 (GPIO_SD_01)
- net BT_CFG02 is gone; now on net GND: U5.76 (GPIO_SD_00)
- net BT_CFG03 is gone; now on net GND: U5.61 (GPIO_SD_13)
- net EN: no longer names the net of U5.24 (PMIC_ON_REQ)
- no-connect marks 4 -> 5
Other:
- note removed: "0"
- note removed: "00"
- note removed: "01"
- note removed: "02"
- note removed: "1"
- note removed: "BOOT_MODE"
- note removed: "BT_CFG"
- note removed: "Boot from fuses"
- note removed: "Encrypted XIP On"
- note removed: "HyperFlash 3.3V"
- note removed: "MXIC Octal DDR"
- note removed: "Micron Octal DDR"
- note removed: "Reserved"
- note removed: "Serial downloader"
- moved on the sheet: C10, C11, C12, C14, C16, C17, C18, C19, C21, C22, C23, C24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
